File: pcb/plaid.kicad_pcb (KiCad board)
At the start: 2 copper layers, 228 x 98 mm, 139 parts, among them J1 USB_OTG, J2 AVR_ISP_6, J3 Conn_01x04, J4 GS2, J5 GS2, SW1 SW_Push, SW10 SW_Push, SW11 SW_Push, SW12 SW_Push, SW13 SW_Push, SW14 SW_Push, SW15 SW_Push, SW16 SW_Push, SW17 SW_Push, SW18 SW_Push, SW19 SW_Push, SW2 SW_Push, SW20 SW_Push, SW21 SW_Push, SW22 SW_Push, SW23 SW_Push, SW24 SW_Push, SW25 SW_Push, SW26 SW_Push, SW27 SW_Push, SW28 SW_Push, SW29 SW_Push, SW3 SW_Push, SW30 SW_Push, SW31 SW_Push, SW32 SW_Push, SW33 SW_Push, SW34 SW_Push, SW35 SW_Push, SW36 SW_Push, SW37 SW_Push, SW38 SW_Push, SW39 SW_Push, SW4 SW_Push, SW40 SW_Push, SW41 SW_Push, SW42 SW_Push, SW43 SW_Push, SW44 SW_Push, SW45 SW_Push, SW46 SW_Push, SW47 SW_Push, SW48 SW_Push, SW49 SW_Push, SW5 SW_Push, SW50 RESET, SW51 BOOT, SW6 SW_Push, SW7 SW_Push, SW8 SW_Push, SW9 SW_Push, U1 ATMEGA328-PU, Y1 16MHz

Commit message: switched footprints to MX/Alps compatible ones
Parts:
- SW1, SW10, SW11, SW12, SW13, SW14, SW15, SW16, SW17, SW18, SW19, SW2, SW20, SW21, SW22, SW23, SW24, SW25, SW26, SW27, SW28, SW29, SW3, SW30, SW31, SW32, SW33, SW34, SW35, SW36, SW37, SW38, SW39, SW4, SW40, SW41, SW42, SW43, SW44, SW45, SW46, SW47, SW48, SW5, SW6, SW7, SW8, SW9: footprint SMKJP:SW_Cherry_MX1A_1.00u_PCB -> MX_Alps_Hybrid:MX-1U-NoLED_edit_no_Fsilk
- SW49: footprint SMKJP:SW_Cherry_MX1A_2.0U_PCB_universal_center -> MX_Alps_Hybrid:MX-2U-ReversedStabilizers-NoLED
Routing:
- net Net-(D12-Pad2): track 100.6 -> 105.2 mm
- net Net-(D35-Pad2): track 119.3 -> 122.1 mm
- net /COL11: track 103.9 -> 101.5 mm
- net Net-(D47-Pad2): track 140.5 -> 142.7 mm
- net Net-(D37-Pad2): track 85.9 -> 84.0 mm
- net Net-(D25-Pad2): track 62.6 -> 60.7 mm
- net Net-(D13-Pad2): track 39.4 -> 37.4 mm
- net /COL5: track 158.5 -> 160.3 mm
- net Net-(D34-Pad2): track 107.3 -> 108.8 mm
- net /COL10: track 85.1 -> 86.4 mm
- net Net-(D46-Pad2): track 128.7 -> 129.8 mm
- net /COL8: track 81.6 -> 80.8 mm
- net Net-(D11-Pad2): track 91.9 -> 91.1 mm
- net Net-(D6-Pad2): track 51.0 -> 51.6 mm
